File: eagle/binw2.brd (EAGLE design)
At the start: 16.9 x 33 mm, 23 parts, among them IC1 ATTINY13V-10SU

Commit message: I don't even know :)
Parts:
- added R6: 10K, resistor:R0805
- added R7: 22K, resistor:R0805
- added S1, S2: DTS-6, switch-tact:DTS-6
Connections:
- new net N$12: R6.2, S1.3
- new net N$3: R7.2, S2.3
- net N$5: now also S1.1, S2.1
- net VCC: now also R6.1, R7.1
Routing:
- net N$5: track 27.1 -> 26.5 mm
Changed lines of the file:
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@@
 <?xml version="1.0" encoding="utf-8"?>
 <!DOCTYPE eagle SYSTEM "eagle.dtd">
-<eagle version="6.0">
+<eagle version="7.6.0">
 <drawing>
 <settings>
@@
 <layer number="97" name="Info" color="7" fill="1" visible="no" active="no"/>
 <layer number="98" name="Guide" color="6" fill="1" visible="no" active="no"/>
+<layer number="99" name="SpiceOrder" color="5" fill="1" visible="no" active="no"/>
 <layer number="250" name="Descript" color="3" fill="1" visible="no" active="no"/>
 <layer number="251" name="SMDround" color="12" fill="11" visible="no" active="no"/>
@@
 </class>
 </classes>
-<designrules>
+<designrules name="default">
 <description language="de">&lt;b&gt;EAGLE Design Rules&lt;/b&gt;
 &lt;p&gt;
@@
 <pass name="Default">
 <param name="RoutingGrid" value="0.5mm"/>
+<param name="AutoGrid" value="1"/>
+<param name="Efforts" value="0"/>
+<param name="TopRouterVariant" value="1"/>
 <param name="tpViaShape" value="octagon"/>
 <param name="PrefDir.1" value="*"/>
@@
 <element name="PAD3" library="wirepad" package="1,6/0,8" value="" x="1.77" y="3.81"/>
 <element name="PAD4" library="wirepad" package="1,6/0,8" value="" x="4.77" y="7.27"/>
+<element name="S1" library="switch-tact" package="DTS-6" value="DTS-6" x="-5.4" y="4.6"/>
+<element name="S2" library="switch-tact" package="DTS-6" value="DTS-6" x="-16.1" y="4.6"/>
+<element name="R6" library="resistor" package="R0805" value="10K" x="-19.4" y="-4"/>
+<element name="R7" library="resistor" package="R0805" value="22K" x="-19.4" y="-8"/>
 </elements>
 <signals>
@@
 <wire x1="3" y1="25.5" x2="3.5" y2="26" width="0.2032" layer="1"/>
 <wire x1="3.5" y1="28.5" x2="3.54" y2="28.7" width="0.2032" layer="1"/>
-<wire x1="3" y1="25.5" x2="2.89" y2="25.29" width="0.2032" layer="1"/>
+<wire x1="3" y1="25.5" x2="2.89" y2="25.39" width="0.2032" layer="1"/>
 </signal>
 <signal name="N$5">
-<contactref element="R5" pad="1"/>
 <contactref element="IC1" pad="3"/>
 <wire x1="0.5" y1="3.5" x2="0.5" y2="21" width="0.2032" layer="1"/>
@@
 <wire x1="4.1" y1="2.5" x2="1.5" y2="2.5" width="0.2032" layer="1"/>
 <wire x1="4.6" y1="3" x2="4.1" y2="2.5" width="0.2032" layer="1"/>
-<wire x1="2.5" y1="23.5" x2="2.89" y2="23.59" width="0.2032" layer="1"/>
 <wire x1="4.6" y1="3" x2="5.466" y2="2.955" width="0.2032" layer="1"/>
 <wire x1="0.5" y1="21" x2="2.89" y2="23.39" width="0.2032" layer="1"/>
-<wire x1="2.89" y1="23.39" x2="2.89" y2="23.59" width="0.2032" layer="1"/>
+<contactref element="R5" pad="1"/>
+<contactref element="S2" pad="1"/>
+<contactref element="S1" pad="1"/>
+<wire x1="2.89" y1="23.39" x2="2.89" y2="23.49" width="0" layer="19" extent="1-1"/>
+<wire x1="-8.65" y1="6.85" x2="0.5" y2="3.5" width="0" layer="19" extent="1-1"/>
+<wire x1="-19.35" y1="6.85" x2="-8.65" y2="6.85" width="0" layer="19" extent="1-1"/>
 </signal>
 <signal name="N$6">
@@
 <wire x1="10.75" y1="1.75" x2="11" y2="1.5" width="0.2032" layer="1"/>
 <wire x1="11.5" y1="1.5" x2="11.774" y2="1.675" width="0.2032" layer="1"/>
-<wire x1="13.02" y1="12.93" x2="12.7" y2="13.25" width="0.2032" layer="1"/>
+<wire x1="13.02" y1="12.83" x2="12.7" y2="13.25" width="0.2032" layer="1"/>
 <wire x1="12.7" y1="13.25" x2="11.5" y2="13.25" width="0.2032" layer="1"/>
 <wire x1="7.35" y1="11.75" x2="7.1" y2="12" width="0.2032" layer="1"/>
@@
 <wire x1="6.5" y1="14" x2="6.5" y2="15" width="0.2032" layer="1"/>
 <wire x1="3.5" y1="10" x2="3.54" y2="9.65" width="0.2032" layer="1"/>
-<wire x1="6.5" y1="14" x2="6.7" y2="13.78" width="0.2032" layer="1"/>
+<wire x1="6.5" y1="14" x2="6.6" y2="13.78" width="0.2032" layer="1"/>
 <wire x1="9" y1="16" x2="11.16" y2="16" width="0.2032" layer="1"/>
 <wire x1="8" y1="15" x2="9" y2="16" width="0.2032" layer="1"/>
@@
 <wire x1="6.5" y1="10.75" x2="8" y2="10.75" width="0.2032" layer="1"/>
 <wire x1="6.5" y1="8.5" x2="6.5" y2="10.75" width="0.2032" layer="1"/>
-<wire x1="8.5" y1="13.5" x2="8.4" y2="13.78" width="0.2032" layer="1"/>
+<wire x1="8.5" y1="13.5" x2="8.5" y2="13.78" width="0.2032" layer="1"/>
 <wire x1="7.35" y1="24.45" x2="7.5" y2="24.45" width="0.2032" layer="1"/>
 <wire x1="7.5" y1="24.45" x2="7.5" y2="24.5" width="0.2032" layer="1"/>
 <wire x1="7.5" y1="24.5" x2="8.5" y2="25.5" width="0.2032" layer="1"/>
 <wire x1="8.5" y1="25.5" x2="9" y2="25.5" width="0.2032" layer="1"/>
-<wire x1="8.4" y1="13.78" x2="9.28" y2="13.78" width="0.2032" layer="1"/>
+<wire x1="8.5" y1="13.78" x2="9.28" y2="13.78" width="0.2032" layer="1"/>
 <wire x1="9.28" y1="13.78" x2="10" y2="14.5" width="0.2032" layer="1"/>
 <wire x1="6.5" y1="8.5" x2="9.5" y2="8.5" width="0.2032" layer="1"/>
@@
 <wire x1="11" y1="20" x2="11" y2="18.5" width="0.2032" layer="1"/>
 <wire x1="11" y1="18.5" x2="11.16" y2="18.1" width="0.2032" layer="1"/>
-<wire x1="11" y1="20" x2="10.65" y2="20.09" width="0.2032" layer="1"/>
+<wire x1="11" y1="20" x2="10.55" y2="20.09" width="0.2032" layer="1"/>
 <wire x1="12.2" y1="23.4" x2="11.5" y2="24" width="0.2032" layer="1"/>
 <wire x1="12.2" y1="21.3" x2="12.2" y2="23.4" width="0.2032" layer="1"/>
@@
 <wire x1="16.5" y1="17" x2="14" y2="17" width="0.2032" layer="1"/>
 <wire x1="15" y1="12" x2="14.97" y2="11.75" width="0.2032" layer="1"/>
-<wire x1="10.65" y1="20.09" x2="10.8" y2="20.24" width="0.2032" layer="1"/>
+<wire x1="10.55" y1="20.09" x2="10.8" y2="20.24" width="0.2032" layer="1"/>
 <wire x1="10.8" y1="20.24" x2="10.8" y2="21.3" width="0.2032" layer="1"/>
 <wire x1="10.8" y1="21.3" x2="12.2" y2="21.3" width="0.2032" layer="1"/>
@@
 <wire x1="3.5" y1="7.5" x2="2" y2="9" width="0.2032" layer="1"/>
 <wire x1="3.5" y1="5.5" x2="3.5" y2="7.5" width="0.2032" layer="1"/>
-<wire x1="4.5" y1="19.5" x2="4.89" y2="19.9" width="0.2032" layer="1"/>
+<wire x1="4.5" y1="19.5" x2="4.89" y2="20" width="0.2032" layer="1"/>
 <wire x1="14.97" y1="18.1" x2="14.5" y2="18.1" width="0.2032" layer="1"/>
-<wire x1="4.89" y1="19.9" x2="5.4" y2="19.9" width="0.2032" layer="1"/>
+<wire x1="4.89" y1="20" x2="5.4" y2="19.9" width="0.2032" layer="1"/>
 <wire x1="5.4" y1="19.9" x2="6.5" y2="21" width="0.2032" layer="1"/>
 <wire x1="14.97" y1="18.1" x2="14.97" y2="18.97" width="0.2032" layer="1"/>
@@
 <wire x1="5.5" y1="18.5" x2="5" y2="18.5" width="0.2032" layer="1"/>
 <wire x1="9.5" y1="22.5" x2="5.5" y2="18.5" width="0.2032" layer="1"/>
-<wire x1="5" y1="18.5" x2="4.89" y2="18.2" width="0.2032" layer="1"/>
+<wire x1="5" y1="18.5" x2="4.89" y2="18.1" width="0.2032" layer="1"/>
 <wire x1="5.5" y1="18.5" x2="7" y2="18.5" width="0.2032" layer="1"/>
 <wire x1="7" y1="18.5" x2="7.35" y2="18.1" width="0.2032" layer="1"/>
-<wire x1="5.5" y1="18.5" x2="4.89" y2="18.2" width="0.2032" layer="1"/>
+<wire x1="5.5" y1="18.5" x2="4.89" y2="18.1" width="0.2032" layer="1"/>
 </signal>
 <signal name="N$13">
@@
 <wire x1="12" y1="20" x2="12" y2="15" width="0.2032" layer="1"/>
 <wire x1="7.5" y1="10" x2="7.35" y2="9.65" width="0.2032" layer="1"/>
-<wire x1="12" y1="20" x2="12.35" y2="20.09" width="0.2032" layer="1"/>
+<wire x1="12" y1="20" x2="12.45" y2="20.09" width="0.2032" layer="1"/>
 <wire x1="12.5" y1="20" x2="13.7" y2="21.2" width="0.2032" layer="1"/>
 <wire x1="13.7" y1="21.2" x2="14.5" y2="22" width="0.2032" layer="1"/>
 <wire x1="14.5" y1="22" x2="14.97" y2="22.35" width="0.2032" layer="1"/>
-<wire x1="12.5" y1="20" x2="12.35" y2="20.09" width="0.2032" layer="1"/>
+<wire x1="12.5" y1="20" x2="12.45" y2="20.09" width="0.2032" layer="1"/>
 <wire x1="13.7" y1="24.3" x2="7.5" y2="30.5" width="0.2032" layer="1"/>
 <wire x1="13.7" y1="21.2" x2="13.7" y2="24.3" width="0.2032" layer="1"/>
@@
 <wire x1="13.5" y1="11.5" x2="13.5" y2="10" width="0.2032" layer="1"/>
 <wire x1="14.1" y1="12.15" x2="13.5" y2="11.5" width="0.2032" layer="1"/>
-<wire x1="13.5" y1="15" x2="13.02" y2="14.63" width="0.2032" layer="1"/>
+<wire x1="13.5" y1="15" x2="13.02" y2="14.73" width="0.2032" layer="1"/>
 <wire x1="14.1" y1="12.15" x2="14.1" y2="13.85" width="0.2032" layer="1"/>
 <wire x1="14.1" y1="13.85" x2="13.37" y2="14.63" width="0.2032" layer="1"/>
-<wire x1="13.37" y1="14.63" x2="13.02" y2="14.63" width="0.2032" layer="1"/>
+<wire x1="13.37" y1="14.63" x2="13.02" y2="14.73" width="0.2032" layer="1"/>
 </signal>
 <signal name="N$15">
@@
 <wire x1="12" y1="5.5" x2="11.774" y2="5.485" width="0.2032" layer="1"/>
 <wire x1="12" y1="7" x2="12.27" y2="7.39" width="0.2032" layer="1"/>
+<contactref element="R6" pad="1"/>
+<contactref element="R7" pad="1"/>
+<wire x1="-20.35" y1="-4" x2="-20.35" y2="-8" width="0" layer="19" extent="1-1"/>
+<wire x1="11.774" y1="5.485" x2="-20.35" y2="-4" width="0" layer="19" extent="1-1"/>
 </signal>
 <signal name="GND">
@@
 <wire x1="1.5" y1="7" x2="1.77" y2="7.35" width="0.2032" layer="1"/>
 </signal>
+<signal name="N$3">
+<contactref element="S2" pad="3"/>
+<contactref element="R7" pad="2"/>
+<wire x1="-19.35" y1="2.35" x2="-18.45" y2="-8" width="0" layer="19" extent="1-1"/>
+</signal>
+<signal name="N$12">
+<contactref element="R6" pad="2"/>
+<contactref element="S1" pad="3"/>
+<wire x1="-8.65" y1="2.35" x2="-18.45" y2="-4" width="0" layer="19" extent="1-1"/>
+</signal>
 </signals>
