File: eagle/binw2.sch (EAGLE design)
At the start: 23 parts, among them IC1 ATTINY13V-10SU

Commit message: I don't even know :)
Parts:
- added R6: 10K, resistor:R-US_R0805
- added R7: 22K, resistor:R-US_R0805
- added S1, S2: DTS-6, switch-tact:DTS-6
Connections:
- new net N$12: R6.2, S1.3
- new net N$3: R7.2, S2.3
- net N$5: now also S1.1, S2.1
- net VCC: now also R6.1, R7.1
Other:
- moved on the sheet: R5
Changed lines of the file:
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@@
 <?xml version="1.0" encoding="utf-8"?>
 <!DOCTYPE eagle SYSTEM "eagle.dtd">
-<eagle version="6.0">
+<eagle version="7.6.0">
 <drawing>
 <settings>
@@
 <layer number="97" name="Info" color="7" fill="1" visible="yes" active="yes"/>
 <layer number="98" name="Guide" color="6" fill="1" visible="yes" active="yes"/>
+<layer number="99" name="SpiceOrder" color="5" fill="1" visible="yes" active="yes"/>
 <layer number="250" name="Descript" color="3" fill="1" visible="no" active="no"/>
 <layer number="251" name="SMDround" color="12" fill="11" visible="no" active="no"/>
@@
 <part name="GND1" library="supply1" deviceset="GND" device=""/>
 <part name="P+1" library="supply1" deviceset="VCC" device=""/>
+<part name="S1" library="switch-tact" deviceset="DTS-6" device=""/>
+<part name="S2" library="switch-tact" deviceset="DTS-6" device=""/>
+<part name="R6" library="resistor" deviceset="R-US_" device="R0805" value="10K"/>
+<part name="R7" library="resistor" deviceset="R-US_" device="R0805" value="22K"/>
 </parts>
 <sheets>
@@
 <instance part="R3" gate="G$1" x="83.82" y="45.72"/>
 <instance part="R4" gate="G$1" x="114.3" y="45.72"/>
-<instance part="R5" gate="G$1" x="144.78" y="40.64"/>
+<instance part="R5" gate="G$1" x="139.7" y="53.34" rot="R90"/>
 <instance part="PAD1" gate="P" x="68.58" y="7.62" rot="R90"/>
 <instance part="PAD2" gate="P" x="86.36" y="7.62" rot="R90"/>
@@
 <instance part="GND1" gate="1" x="78.74" y="2.54"/>
 <instance part="P+1" gate="VCC" x="48.26" y="25.4"/>
+<instance part="S1" gate="G$1" x="109.22" y="30.48" rot="R270"/>
+<instance part="S2" gate="G$1" x="132.08" y="30.48" rot="R270"/>
+<instance part="R6" gate="G$1" x="119.38" y="22.86" rot="R90"/>
+<instance part="R7" gate="G$1" x="142.24" y="22.86" rot="R90"/>
 </instances>
 <busses>
@@
 <segment>
 <pinref part="LED13" gate="G$1" pin="C"/>
-<wire x1="144.78" y1="68.58" x2="149.86" y2="68.58" width="0.1524" layer="91"/>
-<wire x1="149.86" y1="68.58" x2="149.86" y2="40.64" width="0.1524" layer="91"/>
+<wire x1="144.78" y1="68.58" x2="139.7" y2="68.58" width="0.1524" layer="91"/>
+<wire x1="139.7" y1="68.58" x2="139.7" y2="58.42" width="0.1524" layer="91"/>
 <pinref part="R5" gate="G$1" pin="2"/>
 </segment>
@@
 <net name="N$5" class="0">
 <segment>
+<pinref part="IC1" gate="G$1" pin="PB4"/>
+<wire x1="81.28" y1="40.64" x2="81.28" y2="38.1" width="0.1524" layer="91"/>
 <pinref part="R5" gate="G$1" pin="1"/>
-<pinref part="IC1" gate="G$1" pin="PB4"/>
-<wire x1="139.7" y1="40.64" x2="81.28" y2="40.64" width="0.1524" layer="91"/>
-<wire x1="81.28" y1="40.64" x2="81.28" y2="38.1" width="0.1524" layer="91"/>
+<wire x1="81.28" y1="40.64" x2="101.6" y2="40.64" width="0.1524" layer="91"/>
+<wire x1="101.6" y1="40.64" x2="124.46" y2="40.64" width="0.1524" layer="91"/>
+<wire x1="124.46" y1="40.64" x2="139.7" y2="40.64" width="0.1524" layer="91"/>
+<wire x1="139.7" y1="40.64" x2="139.7" y2="48.26" width="0.1524" layer="91"/>
+<pinref part="S2" gate="G$1" pin="1"/>
+<wire x1="127" y1="30.48" x2="124.46" y2="30.48" width="0.1524" layer="91"/>
+<wire x1="124.46" y1="30.48" x2="124.46" y2="40.64" width="0.1524" layer="91"/>
+<pinref part="S1" gate="G$1" pin="1"/>
+<wire x1="104.14" y1="30.48" x2="101.6" y2="30.48" width="0.1524" layer="91"/>
+<wire x1="101.6" y1="30.48" x2="101.6" y2="40.64" width="0.1524" layer="91"/>
+<junction x="101.6" y="40.64"/>
+<junction x="124.46" y="40.64"/>
 </segment>
 </net>
@@
 <wire x1="68.58" y1="17.78" x2="68.58" y2="15.24" width="0.1524" layer="91"/>
 <wire x1="68.58" y1="15.24" x2="68.58" y2="10.16" width="0.1524" layer="91"/>
-<wire x1="48.26" y1="15.24" x2="68.58" y2="15.24" width="0.1524" layer="91"/>
+<wire x1="48.26" y1="15.24" x2="53.34" y2="15.24" width="0.1524" layer="91"/>
 <junction x="68.58" y="15.24"/>
+<wire x1="53.34" y1="15.24" x2="68.58" y2="15.24" width="0.1524" layer="91"/>
+<wire x1="53.34" y1="15.24" x2="53.34" y2="-2.54" width="0.1524" layer="91"/>
+<pinref part="R6" gate="G$1" pin="1"/>
+<wire x1="53.34" y1="-2.54" x2="119.38" y2="-2.54" width="0.1524" layer="91"/>
+<wire x1="119.38" y1="-2.54" x2="119.38" y2="17.78" width="0.1524" layer="91"/>
+<junction x="53.34" y="15.24"/>
+<pinref part="R7" gate="G$1" pin="1"/>
+<wire x1="142.24" y1="17.78" x2="142.24" y2="-2.54" width="0.1524" layer="91"/>
+<wire x1="142.24" y1="-2.54" x2="119.38" y2="-2.54" width="0.1524" layer="91"/>
+<junction x="119.38" y="-2.54"/>
 </segment>
 </net>
@@
 </segment>
 </net>
+<net name="N$3" class="0">
+<segment>
+<pinref part="S2" gate="G$1" pin="3"/>
+<pinref part="R7" gate="G$1" pin="2"/>
+<wire x1="137.16" y1="30.48" x2="142.24" y2="30.48" width="0.1524" layer="91"/>
+<wire x1="142.24" y1="30.48" x2="142.24" y2="27.94" width="0.1524" layer="91"/>
+</segment>
+</net>
+<net name="N$12" class="0">
+<segment>
+<pinref part="S1" gate="G$1" pin="3"/>
+<pinref part="R6" gate="G$1" pin="2"/>
+<wire x1="119.38" y1="27.94" x2="119.38" y2="30.48" width="0.1524" layer="91"/>
+<wire x1="119.38" y1="30.48" x2="114.3" y2="30.48" width="0.1524" layer="91"/>
+</segment>
+</net>
